File: PCB/FlexRC/Buttons.kicad_sch (KiCad schematic)
At the start: 36 parts

Commit message: pico_v1
Parts:
- added C19, C20: 100n, Capacitor_SMD:C_1206_3216Metric_Pad1.33x1.80mm_HandSolder, symbol Device:C
- renumbered C1 to C12, C2 to C13, C3 to C14, C4 to C15, C5 to C16, C6 to C17, C7 to C18, C8 to C21, C17 to C22, JOY_R_2 to JOY_R_1, R8 to R13, R9 to R14, R10 to R15, R11 to R16, R12 to R17, R13 to R18, R14 to R19, R1 to R20, R2 to R21, R3 to R22, R4 to R23, R5 to R24, R6 to R25, R7 to R26, R15 to R27, R17 to R28, R16 to R29, R18 to R30
Connections:
- net CH7 is gone; now on net CH6: C22.1, R30.2
- net +3.3V: now also C19.2, C20.2
- net CH6: no longer C21.1, R29.2
- net GND: now also C19.1, C20.1
- new net CH5: C21.1, R29.2
Other:
- company: (none) -> Flex Electronics
- title: (none) -> FlexRC
- moved on the sheet: C12, C13, C14, C15, C16, C17, C18, C21, C22, JOY_L_1, JOY_R_1, R13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
