File: PCB/FlexRC/FlexRC.kicad_sch (KiCad schematic)
At the start: 0 parts

Commit message: 0116
Parts:
- added DS1: SSD1306_128x64, flexrc_footprints:OLED_SSD1306_128x64_Module, symbol flexrc_symbols:OLED_SSD1306_128x64_Module
Connections:
- new net +3V3: DS1.1 (VDD)
- new net GND: DS1.2 (GND)

Commit message: 123
Parts:
- removed DS1: SSD1306_128x64, flexrc_footprints:OLED_SSD1306_128x64_Module, symbol flexrc_symbols:OLED_SSD1306_128x64_Module
Other:
- added sheet Buttons_Joys (Buttons.kicad_sch)
- added sheet MCU (MCU.kicad_sch)
- added sheet Power (Power.kicad_sch)
- added sheet RGBs (RGBs.kicad_sch)
- added sheet Radio (Radio.kicad_sch)

Commit message: pico_v1
Other:
- sheet MCU renamed MCU_RADIO_OLED
- removed sheet Radio
- company: (none) -> Flex Electronics
- title: (none) -> FlexRC
Changed lines of the file:
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@@
 	(generator_version "9.0")
 	(paper "A4")
+	(title_block
+		(title "FlexRC")
+		(date "2026-03-06")
+		(rev "V1")
+		(company "Flex Electronics")
+		(comment 1 "Luke")
+		(comment 2 "https://github.com/LukeSky91/FlexRC")
+	)
 	(sheet
 		(at 25.4 63.5)
@@
 			(color 0 0 0 0.0000)
 		)
-		(property "Sheetname" "MCU"
+		(property "Sheetname" "MCU_RADIO_OLED"
 			(at 25.4 62.7884 0)
 			(effects
@@
 	)
 	(sheet
-		(at 25.4 101.6)
-		(size 38.1 25.4)
-		(exclude_from_sim no)
-		(in_bom yes)
-		(on_board yes)
-		(dnp no)
-		(fields_autoplaced yes)
-		(stroke
-			(width 0.1524)
-			(type solid)
-		)
-		(fill
-			(color 0 0 0 0.0000)
-		)
-		(property "Sheetname" "Radio"
-			(at 25.4 100.8884 0)
-			(effects
-				(font
-					(size 1.27 1.27)
-				)
-				(justify left bottom)
-			)
-		)
-		(property "Sheetfile" "Radio.kicad_sch"
-			(at 25.4 127.5846 0)
-			(effects
-				(font
-					(size 1.27 1.27)
-				)
-				(justify left top)
-			)
-		)
-		(instances
-			(project "FlexRC"
-				(path "/0116ad82-ac95-4a03-bd4e-94de3191d2e0"
-					(page "4")
-				)
-			)
-		)
-	)
-	(sheet
 		(at 76.2 63.5)
 		(size 38.1 25.4)
@@
 			(project "FlexRC"
 				(path "/0116ad82-ac95-4a03-bd4e-94de3191d2e0"
-					(page "9")
+					(page "5")
 				)
 			)
@@
 			(project "FlexRC"
 				(path "/0116ad82-ac95-4a03-bd4e-94de3191d2e0"
-					(page "8")
+					(page "4")
 				)
 			)
