File: PCB/FlexRC/MCU.kicad_sch (KiCad schematic)
At the start: 2 parts

Commit message: pico_v1
Parts:
- added C10: 10u, Capacitor_THT:CP_Radial_Tantal_D5.0mm_P2.50mm, symbol Device:C_Polarized
- added C11, C6, C8, C9: 100n, Capacitor_SMD:C_1206_3216Metric_Pad1.33x1.80mm_HandSolder, symbol Device:C
- added C5, C7: 100u, Capacitor_THT:CP_Radial_Tantal_D6.0mm_P2.50mm, symbol Device:C_Polarized
- added R10, R11: 35R, Resistor_SMD:R_1206_3216Metric_Pad1.30x1.75mm_HandSolder, symbol Device:R
- added R12: 1k, Resistor_SMD:R_1206_3216Metric_Pad1.30x1.75mm_HandSolder, symbol Device:R
- added R6, R7: 4k7, Resistor_SMD:R_1206_3216Metric_Pad1.30x1.75mm_HandSolder, symbol Device:R
- added R8: photoR, flexrc_footprints:photoResistor, symbol Device:R_Photo
- added R9: 10k, Resistor_SMD:R_1206_3216Metric_Pad1.30x1.75mm_HandSolder, symbol Device:R
- added TX1: NRF24L01_Breakout, flexrc_footprints:nRF24L01_Breakout, symbol RF:NRF24L01_Breakout
- renumbered DS2 to DS1
Connections:
- net +5V is gone; now on net +3.3V: A1.39 (VSYS)
- net +3.3V: now also C10.1, C11.1, C5.1, C6.1, C7.1, C8.1, R6.2, R7.2, R8.1, TX1.2 (VCC)
- net CH7: now also C9.1, R12.2
- net GND: now also C10.2, C11.2, C5.2, C6.2, C7.2, C8.2, C9.2, R9.2, TX1.1 (GND)
- net GP17: now also R10.1, R7.1; no longer DS1.3 (SCL)
- net GP18: now also R11.1, R6.1; no longer DS1.4 (SDA)
- net GP34: now also TX1.5 (SCK)
- net GP35: now also TX1.6 (MOSI)
- net GP36: now also TX1.7 (MISO)
- net GP37: now also TX1.4 (~{CSN})
- net GP38: now also TX1.3 (CE)
- net CH8: now reaches A1.34 (ADC1_CH8_GP9)
- new net: DS1.3 (SCL), R10.2
- new net: R12.1, R8.2, R9.1
- new net: DS1.4 (SDA), R11.2
Other:
- note added: "PHOTO R"
- company: (none) -> Flex Electronics
- title: (none) -> FlexRC
- moved on the sheet: A1
