File: PCB/FlexRC/Power.kicad_sch (KiCad schematic)
At the start: 15 parts, among them U1 SparkFun 3.3V

Commit message: pico_v1
Parts:
- removed J_BATT_OUT: BATTERY_OUTPUT, TestPoint:TestPoint_Bridge_Pitch2.54mm_Drill1.0mm, symbol Connector:Conn_01x02_Pin
- added C3: 220u, Capacitor_THT:CP_Radial_Tantal_D6.0mm_P2.50mm, symbol Device:C_Polarized
- added J1: Conn_01x02, flexrc_footprints:2pin_header, symbol Connector_Generic:Conn_01x02
- added SW_PWR_1: SW_SPDT, flexrc_footprints:power_switch, symbol Switch:SW_SPDT
- added U2: 5V_mini_buck, flexrc_footprints:5V_mini_buck, symbol flexrc_symbols:5V_buck
- C1: renamed from C19; footprint Capacitor_THT:CP_Radial_D10.0mm_P3.80mm -> Capacitor_THT:CP_Radial_Tantal_D6.0mm_P2.50mm
- C2: renamed from C20; footprint Capacitor_SMD:C_1206_3216Metric_Pad1.33x1.80mm_HandSolder -> Capacitor_THT:C_Radial_D5.0mm_H5.0mm_P2.00mm
- C4: renamed from C18; footprint Capacitor_SMD:C_1206_3216Metric_Pad1.33x1.80mm_HandSolder -> Capacitor_THT:C_Radial_D5.0mm_H5.0mm_P2.00mm
- renumbered R21 to R1, R22 to R2, R23 to R3, R24 to R4, R25 to R5
Connections:
- net +3.3V: now also C3.1
- net +8V: now also C1.1, C2.1, F1.2, U2.1 (VIN)
- net GND: now also C1.2, C2.2, C3.2, J1.1 (Pin_1), U2.2 (GND), U2.4 (GND)
- net at BT1.1 (+), Balancer1.1 (B+): now also BT1.2 (-), BT2.1 (+), BT2.2 (-), Balancer1.2 (BM), Balancer1.3 (B-); no longer Charg1.1 (B+)
- net at Balancer1.4 (P+): now also Charg1.1 (B+)
- net at Balancer1.5 (P-): now also Charg1.3 (B-)
- net at F1.1: now also SW_PWR_1.3 (C)
- net CH5 renamed CH8
- new net: J1.2 (Pin_2), SW_PWR_1.2 (B)
- new net +5V: U2.3 (OUT)
- now unconnected: Charg1.2 (BM)
- no-connect marks 2 -> 4
Other:
- company: (none) -> Flex Electronics
- title: (none) -> FlexRC
- moved on the sheet: BT1, BT2, Balancer1, C1, C2, C4, Charg1, F1, R1, R2, R3, R4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
