File: PCB/FlexRC/RGBs.kicad_sch (KiCad schematic)
At the start: 11 parts

Commit message: pico_v1
Parts:
- added R31: 220R, Resistor_SMD:R_1206_3216Metric_Pad1.30x1.75mm_HandSolder, symbol Device:R
- added U3: 74AHCT1G125, Package_TO_SOT_SMD:SOT-353_SC-70-5_Handsoldering, symbol 74xGxx:74AHCT1G125
- C23: renamed from C10; value 470u -> 220u; footprint Capacitor_THT:CP_Radial_D10.0mm_P3.80mm -> Capacitor_THT:CP_Radial_Tantal_D6.0mm_P2.50mm
- renumbered C11 to C24, C14 to C25, C12 to C26, C15 to C27, C13 to C28, D4 to D2, D2 to D3, D5 to D4, D3 to D5
Connections:
- net D1_out: now also D2.4 (DIN); no longer D3.4 (DIN)
- net D2_out: now also D2.2 (DOUT), D3.4 (DIN); no longer D3.2 (DOUT), D5.4 (DIN)
- net D3_out: now also D3.2 (DOUT), D4.4 (DIN); no longer D2.4 (DIN), D5.2 (DOUT)
- net D4_out: now also D4.2 (DOUT), D5.4 (DIN); no longer D2.2 (DOUT), D4.4 (DIN)
- net GND: now also U3.1, U3.3 (GND)
- net GP39: now also R31.1; no longer D1.4 (DIN)
- net +3.3V renamed +5V
- net +5V: now also U3.5 (VCC)
- new net: R31.2, U3.2
- new net GP39_LS: D1.4 (DIN), U3.4
Other:
- company: (none) -> Flex Electronics
- title: (none) -> FlexRC
- moved on the sheet: C23, C24, C25, C26, C27, C28, D1, D2, D3, D4, D5
